Commit message: Disable mimic joints (isaac bug!)

File: source/ur10e_sim2real/ur10e_sim2real/robots/ur10e/ur10e_with_hande.urdf (robot description, URDF)
Before this commit: robot ur10e_with_hande, 18 links, 17 joints
Joints:
- joint robotiq_hande_right_finger_joint: mimic joint=robotiq_hande_left_finger_joint multiplier=1 offset=0 -> (none)
